Commit message: add robot stand and working table meshes, fix robot base origin

File: ur5e_hande_description/urdf/ur5e_hande.urdf.xacro (robot description, xacro)
@@ -15,5 +15,52 @@
   <xacro:include filename="$(find ur_description)/urdf/ur_macro.xacro"/>
   <xacro:include filename="$(find ur5e_hande_description)/urdf/robotiq_hande_macro.urdf.xacro"/>
+  <!-- World -->
   <link name="world"/>
+  <!-- Working Table -->
+  <link name="working_table">
+    <visual>
+      <origin xyz="0 0 0" rpy="0 0 0"/>
+      <geometry>
+        <mesh filename="package://ur5e_hande_description/meshes/Working_table.stl"/>
+      </geometry>
+      <material name="table_color">
+        <color rgba="0.6 0.4 0.2 1.0"/>
+      </material>
+    </visual>
+    <collision>
+      <origin xyz="0 0 0" rpy="0 0 0"/>
+      <geometry>
+        <mesh filename="package://ur5e_hande_description/meshes/Working_table.stl"/>
+      </geometry>
+    </collision>
+  </link>
+  <joint name="world_to_table" type="fixed">
+    <origin xyz="0 0.75 0" rpy="0 0 0"/>
+    <parent link="world"/>
+    <child link="working_table"/>
+  </joint>
+  <!-- Robot Stand -->
+  <link name="robot_stand">
+    <visual>
+      <origin xyz="0 0 0" rpy="0 0 0"/>
+      <geometry>
+        <mesh filename="package://ur5e_hande_description/meshes/robot_stand.stl"/>
+      </geometry>
+      <material name="stand_color">
+        <color rgba="0.3 0.3 0.3 1.0"/>
+      </material>
+    </visual>
+    <collision>
+      <origin xyz="0 0 0" rpy="0 0 0"/>
+      <geometry>
+        <mesh filename="package://ur5e_hande_description/meshes/robot_stand.stl"/>
+      </geometry>
+    </collision>
+  </link>
+  <joint name="world_to_stand" type="fixed">
+    <origin xyz="0 0 0" rpy="0 0 0"/>
+    <parent link="world"/>
+    <child link="robot_stand"/>
+  </joint>
   <xacro:if value="$(arg sim_gazebo)">
     <link name="ground_plane">
@@ -37,5 +84,5 @@
     name="ur"
     tf_prefix=""
-    parent="world"
+    parent="robot_stand"
     joint_limits_parameters_file="$(find ur_description)/config/$(arg ur_type)/joint_limits.yaml"
     kinematics_parameters_file="$(find ur_description)/config/$(arg ur_type)/default_kinematics.yaml"
@@ -69,5 +116,5 @@
     script_sender_port="$(arg script_sender_port)"
     trajectory_port="$(arg trajectory_port)">
-    <origin xyz="0 0 0" rpy="0 0 0"/>
+    <origin xyz="0 0.235 0.87" rpy="0 0 0"/>
   </xacro:ur_robot>
   <xacro:robotiq_hande_gripper
